Commit message: make finger joint movable + remove block collision

File: assets/panda_xacro/hand.xacro (robot description, xacro)
@@ -90,5 +90,4 @@
       <axis xyz="0 -1 0"/>
       <limit effort="20" lower="0.0" upper="0.04" velocity="0.2"/>
-      <mimic joint="${ns}_finger_joint1" />
       <!-- Gazebo adaptation: dampening-->
       <dynamics damping="${joint_damping}"/>
